File: hardware/power_board/kicad/nibbles_power_board.kicad_sch (KiCad schematic)
At the start: 0 parts

Commit message: Power board: one-sheet schematic drawn as wired blocks, net classes, layout in progress
- KiCad schematic merged into one page; the ideal diodes (U9/Q9, U3/Q5,
  U4/Q6), the eFuse path (U5, bulk caps, shunt R29 and INA226, J3/F1, J5)
  and the 5 V buck (U7) are now wired pin to pin instead of label to
  label. Same netlist; ITIMER, ILIM, IMON and RETRY_DLY now use KiCad's
  automatic net names (renamed to match in the board).
- The KiCad files are now the master copy for the power board; the
  generator refuses a board with tracks.
- Net classes for both boards (Power 5 mm / 3 mm, Supply 1 mm) and
  pre-defined track and via sizes in the generator.
- Placement, routing and pours on the power board so far.

Co-Authored-By: Claude Opus 5.5 <noreply@anthropic.com>
Parts:
- added C30, C31, C38, C47, C48: 0.1uF, Capacitor_SMD:C_0603_1608Metric, symbol nibbles:C
- added C32, C33: 220uF 25V polymer, Capacitor_SMD:CP_Elec_6.3x9.9, symbol nibbles:C
- added C34: 10uF 25V, Capacitor_SMD:C_0805_2012Metric, symbol nibbles:C
- added C35: 10nF (TBD), Capacitor_SMD:C_0603_1608Metric, symbol nibbles:C
- added C36: 100nF (TBD), Capacitor_SMD:C_0603_1608Metric, symbol nibbles:C
- added C37: 22nF (TBD), Capacitor_SMD:C_0603_1608Metric, symbol nibbles:C
- added C40, C41: 10uF 35V, Capacitor_SMD:C_1206_3216Metric, symbol nibbles:C
- added C42: 0.1uF 35V, Capacitor_SMD:C_0603_1608Metric, symbol nibbles:C
- added C43: 100nF, Capacitor_SMD:C_0603_1608Metric, symbol nibbles:C
- added C44, C45: 22uF 10V, Capacitor_SMD:C_0805_2012Metric, symbol nibbles:C
- added C46: 10nF, Capacitor_SMD:C_0603_1608Metric, symbol nibbles:C
- added D2: SMBJ18A, Diode_SMD:D_SMB, symbol nibbles:D
- added D3, D4: TPD1E10B06DPYR, Diode_SMD:D_0402_1005Metric, symbol nibbles:D
- added F1: 15A, Fuse:Fuse_1206_3216Metric, symbol nibbles:FUSE
- added J10: XT30 (charger port: input), Connector_AMASS:AMASS_XT30PW-M_1x02_P2.50mm_Horizontal, symbol nibbles:CONN2_XT30
- added J11: XT30 (charger port: battery), Connector_AMASS:AMASS_XT30PW-M_1x02_P2.50mm_Horizontal, symbol nibbles:CONN2_XT30
- added J12: JST-GH 6 (charger port: I2C), Connector_JST:JST_GH_SM06B-GHS-TB_1x06-1MP_P1.25mm_Horizontal, symbol nibbles:CONN6
- added J2: XT30PW-M (dock power, from the LEMO), Connector_AMASS:AMASS_XT30PW-M_1x02_P2.50mm_Horizontal, symbol nibbles:CONN2_XT30
- added J3: XT30 (pack, from 4S BMS), Connector_AMASS:AMASS_XT30PW-M_1x02_P2.50mm_Horizontal, symbol nibbles:CONN2_XT30
- added J5: XT30 (to the 5 V lighting converter), Connector_AMASS:AMASS_XT30PW-M_1x02_P2.50mm_Horizontal, symbol nibbles:CONN2_XT30
- added J6: To the base board (JST-GH 8), Connector_JST:JST_GH_SM08B-GHS-TB_1x08-1MP_P1.25mm_Horizontal, symbol nibbles:CONN8
- added J7: S3B-PH-K-S (dock data, from the LEMO), Connector_JST:JST_PH_S3B-PH-K_1x03_P2.00mm_Horizontal, symbol nibbles:CONN3
- added J8: S2B-PH-K-S (dock LED, panel), Connector_JST:JST_PH_S2B-PH-K_1x02_P2.00mm_Horizontal, symbol nibbles:CONN2_PH2
- added J9: JST-GH 6 (keypad port: I2C), Connector_JST:JST_GH_SM06B-GHS-TB_1x06-1MP_P1.25mm_Horizontal, symbol nibbles:CONN6
- added L2: 6.8uH Isat>=4A, Inductor_SMD:L_Sunlord_MWSA0603S, symbol nibbles:L
- added Q5, Q6, Q9: 30V N-FET >= 15 A, Package_SO:ONSemi_SO-8FL_488AA, symbol nibbles:NMOS_SO8FL
- added Q7, Q8: 2N7002, Package_TO_SOT_SMD:SOT-23, symbol nibbles:NMOS_SOT23
- added R16, R28: 10k, Resistor_SMD:R_0603_1608Metric, symbol nibbles:R
- added R20, R21, R35: 1M, Resistor_SMD:R_0603_1608Metric, symbol nibbles:R
- added R22, R25, R5: 100k, Resistor_SMD:R_0603_1608Metric, symbol nibbles:R
- added R23: 86.6k 1%, Resistor_SMD:R_0603_1608Metric, symbol nibbles:R
- added R24, R31: 10k 1%, Resistor_SMD:R_0603_1608Metric, symbol nibbles:R
- added R26: 130 1%, Resistor_SMD:R_0603_1608Metric, symbol nibbles:R
- added R27: TBD (IMON), Resistor_SMD:R_0603_1608Metric, symbol nibbles:R
- added R29: 2 mOhm 2512 3W, Resistor_SMD:R_2512_6332Metric, symbol nibbles:R
- added R3, R4: 1k, Resistor_SMD:R_0603_1608Metric, symbol nibbles:R
- added R30: 52.3k 1%, Resistor_SMD:R_0603_1608Metric, symbol nibbles:R
- added R32, R33: 4.7k, Resistor_SMD:R_0603_1608Metric, symbol nibbles:R
- added R36: 7.5k, Resistor_SMD:R_0603_1608Metric, symbol nibbles:R
- added U3: LM74700-Q1 (dock), nibbles_ti:DBV0006A_N, symbol nibbles:LM74700
- added U4: LM74700-Q1 (pack), nibbles_ti:DBV0006A_N, symbol nibbles:LM74700
- added U5: TPS259827ONRGET, nibbles_ti:RGE24_2P5XP85X1P45_TEX, symbol nibbles:TPS25982
- added U6: INA226AIDGSR, nibbles_ti:VSSOP10_DGS_TEX, symbol nibbles:INA228
- added U7: TPS62933DRLR, nibbles_ti:SOT_33DRLR_TEX, symbol nibbles:TPS62933
- added U8: TCA9534PWR, nibbles_ti:PW0016A-MFG, symbol nibbles:TCA9534
- added U9: LM74700-Q1 (LEMO), nibbles_ti:DBV0006A_N, symbol nibbles:LM74700
Connections:
- new net: C35.1, U5.7 (ITIMER)
- new net: C36.1, U5.10 (RETRY_DLY)
- new net: R26.1, U5.8 (ILIM)
- new net: R27.1, U5.9 (IMON)
- new net +3V3: C38.1, C47.1, J12.2, J6.3, J9.2, R16.2, R28.2, R32.2, R33.2, U6.6 (VS), U8.16 (VCC)
- new net +5V: C44.1, C45.1, J12.6, J6.1, J9.6, L2.2, R30.1
- new net BUCK_BST: C43.1, U7.6 (BST)
- new net BUCK_FB: R30.2, R31.1, U7.8 (FB)
- new net BUCK_SS: C46.1, U7.7 (SS)
- new net BUCK_SW: C43.2, L2.1, U7.5 (SW)
- new net DOCK_DATA_RAW: D3.1 (C), J7.1, R3.1
- new net DOCK_DET: J6.8, R4.2, R5.1
- new net DOCK_DET_RAW: D4.1 (C), J7.2, R4.1
- new net DOCK_LED: J8.1, R36.2
- new net DOCK_RAW: C48.2, D2.1 (C), J2.2 (1), Q9.1 (S), Q9.2 (S), Q9.3 (S), R35.1, U9.6 (ANODE)
- new net DOCK_UART: J6.7, R3.2
- new net DOCK_VIN: C30.2, J10.2 (1), Q5.1 (S), Q5.2 (S), Q5.3 (S), Q9.5 (D), R20.1, R36.1, U3.6 (ANODE), U9.4 (CATHODE)
- new net EFUSE_DVDT: C37.1, U5.15 (DVDT)
- new net EFUSE_EN: Q8.3 (D), R23.2, R24.1, U5.6 (EN/UVLO)
- new net EFUSE_OUT: C32.1, C33.1, R29.1, U5.17 (OUT_2), U5.18 (OUT_3), U5.19 (OUT_4), U5.20 (OUT_5), U5.21 (OUT_6), U5.22 (OUT_7), U5.23 (OUT_8), U5.24 (OUT), U6.10 (IN+)
- new net EFUSE_PG: R28.1, U5.13 (PG), U8.7 (P3)
- new net EN_DOCK: R20.2, U3.3 (EN)
- new net EN_LEMO: R35.2, U9.3 (EN)
- new net EN_PACK: Q7.3 (D), R21.2, U4.3 (EN)
- new net GATE_DOCK: Q5.4 (G), U3.5 (GATE)
- new net GATE_LEMO: Q9.4 (G), U9.5 (GATE)
- new net GATE_PACK: Q6.4 (G), U4.5 (GATE)
- new net GND: C32.2, C33.2, C34.2, C35.2, C36.2, C37.2, C38.2, C40.2, C41.2, C42.2, C44.2, C45.2, C46.2, C47.2, D2.2 (A), D3.2 (A), D4.2 (A), J10.1 (2), J11.1 (2), J12.1, J2.1 (2), J3.1 (2), J5.1 (2), J6.2, J7.3, J8.2, J9.1, Q7.2 (S), Q8.2 (S), R22.2, R24.2, R25.2, R26.2, R27.2, R31.2, R5.2, U3.2 (GND), U4.2 (GND), U5.11 (NRETRY), U5.12 (LDSTRT), U5.14 (GND), U5.26 (EPAD), U5.4 (GND_2), U5.5 (GND_3), U6.1 (A1), U6.2 (A0), U6.7 (GND), U7.4 (GND), U8.1 (A0), U8.2 (A1), U8.3 (A2), U8.8 (GND), U9.2 (GND)
- new net LIGHT_BUS: C34.1, C40.1, C41.1, C42.1, Q5.5 (D), Q6.5 (D), R23.1, U3.4 (CATHODE), U4.4 (CATHODE), U5.1 (IN_2), U5.16 (IN), U5.2 (IN_3), U5.25 (EPAD_2), U5.3 (IN_4), U7.3 (VIN)
- new net LIGHT_OFF: Q8.1 (G), R25.1, U8.4 (P0)
- new net LIGHT_OUT: J5.2 (1), R29.2, U6.8 (VBUS), U6.9 (IN-)
- new net PACK_F: C31.2, F1.2, J11.2 (1), Q6.1 (S), Q6.2 (S), Q6.3 (S), R21.1, U4.6 (ANODE)
- new net PACK_OFF: Q7.1 (G), R22.1, U8.5 (P1)
- new net PACK_RAW: F1.1, J3.2 (1)
- new net PWR_INT: J12.5, J6.6, J9.5, R16.1, U6.3 (ALERT), U8.13 (INT_N)
- new net PWR_SCL: J12.4, J6.5, J9.4, R33.1, U6.5 (SCL), U8.14 (SCL)
- new net PWR_SDA: J12.3, J6.4, J9.3, R32.1, U6.4 (SDA), U8.15 (SDA)
- new net VCAP_DOCK: C30.1, U3.1 (VCAP)
- new net VCAP_LEMO: C48.1, U9.1 (VCAP)
- new net VCAP_PACK: C31.1, U4.1 (VCAP)
- no-connect marks 0 -> 7
Other:
- removed sheet Inputs
- removed sheet Lighting
- removed sheet Logic
- note added: "1 Input: dock (LEMO)"
- note added: "2 Lighting path: ideal diodes, eFuse, INA228"
- note added: "3 Logic: 5 V for the base, I/O expander, ports"
- note added: "4 SDA, 5 SCL, 6 INT (open-drain, shared by everything on the bus), 7 dock UART, 8 dock detect."
- note added: "5 V, 3 A max, 500 kHz (RT open), FB 52.3k/10k = 4.98 V. L2 6.8 uH is a starting point (datasheet's inductor table)."
- note added: "Charger port: J10 (XT30, DOCK_VIN out to the charger), J11 (XT30, the charger's battery output into PACK_F),"
- note added: "Dock: the LEMO 1K.308 sits in the enclosure wall and is wired to this board: J2 (XT30) takes its battery"
- note added: "ILIM 130R = about 11.3 A (datasheet: 300R = 5 A, 182R = 8.1 A, 100R = 14.7 A). UVLO 86.6k/10k: on at 11.6 V, off at 10.6 V."
- note added: "INA228 on the output: 2 mOhm shunt, address 0x40 (A0 = A1 = GND); its ALERT shares PWR_INT."
- note added: "ITIMER, RETRY_DLY and dVdt values are starting points: check against the datasheet for the converter's input capacitance."
- note added: "J12 (JST-GH 6: 1 GND, 2 +3V3, 3 SDA, 4 SCL, 5 INT, 6 +5V). Plan B: last year's 60 W + 140 W USB-C modules on J10/J11."
- note added: "J8: a panel LED (with leads, no resistor) lit whenever the dock supplies power, firmware or not (~1-2 mA)."
- note added: "Keypad port: J9, the same JST-GH 6 pinout (the keypad's expander shares INT). Leave the Waveshare battery header empty."
- note added: "LEMO, not the bulk caps: C32/C33 sit behind the eFuse (EFUSE_OUT), which ramps them up (dVdt), and hold up the"
- note added: "LIGHT_BUS has only small ceramics, so plugging a live dock into a switched-off shark charges ~30 uF through the"
- note added: "LIGHT_OFF from the expander turns the lights off; defaults to on, so the lights work without the base."
- note added: "Pack: off-the-shelf 4S BMS on the cells, the main power switch in its lead, XT30 to J3; F1 protects lights and charging."
- note added: "Pole-base power board: dock (LEMO) input, ideal-diode lighting path with eFuse and INA226, 5 V for the base board, I/O expander, charger and keypad ports. Design notes are with each section."
- note added: "Power I2C (BQ25798 0x6B, INA228 0x40, TCA9534 0x20, keypad 0x21-0x27) on its own bus from the Waveshare board;"
- note added: "TCA9534 at 0x20 (A0-A2 = GND): P0 LIGHT_OFF, P1 PACK_OFF (outputs); P3 EFUSE_PG (input); P2, P4-P7 spare."
- note added: "TPS62933 from LIGHT_BUS (dock or pack, 11-16.8 V; not the charger, so the base runs without a charger board):"
- note added: "TVS: SMBJ18A on the dock input (16.8 V max), clamping under the 30 V FETs."
- note added: "The LEMO is the only power input: the dock, or a separate USB-C PD to LEMO charging dongle at home."
- note added: "The pack's can be switched off (PACK_OFF) while the dock runs the lights; its FET's body diode still holds the bus"
- note added: "Two LM74700 ideal diodes OR the dock and the internal pack onto LIGHT_BUS. The dock's is always on."
- note added: "U9/Q9: ideal diode right after the LEMO, so no current ever leaves the shark through it (the pack, the charger,"
- note added: "Unused refs: J1, U1, D1, R1, C1, Q1-Q4, R34 (an earlier USB-C input), J4 and everything on U2 (the charger board)."
- note added: "converter's input while the ideal diodes switch between dock and pack."
- note added: "eFuse TPS259827ONRGE: no overvoltage lockout (the pack and dock reach 16.8 V), circuit breaker."
- note added: "if the dock is pulled, until the base turns it back on. Defaults to on."
- note added: "or plan B's USB-C modules feeding back into the dock). U3/Q5 in section 2 is the dock's separate OR diode into"
- note added: "pins (LEMO 1-3 +, 4-6 ground), J7 (JST-PH 3) its data (LEMO 7, UART to the base), dock detect (8) and a ground."
- note added: "pull-ups here. J6 to the Waveshare ESP32-S3-Touch-LCD-3.49 V2: 1 +5V out, 2 GND, 3 +3V3 in (pull-ups and logic),"
- note added: "the lights: without it, the pack would feed the charger's input through LIGHT_BUS."
- note removed: "Pole-base power board: dock (LEMO) input, ideal-diode lighting path with eFuse and INA226, 5 V for the base board, I/O expander, charger and keypad ports. Design notes are on each sheet."
- title: Nibbles pole-base power board -> Nibbles power board
