File: hardware/charger_board/kicad/1_charger.kicad_sch (KiCad schematic)
At the start: 34 parts, among them J21 XT30 (from the power board: i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, J22 XT30 (to the power board: bat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, J23 JST-GH 6 (to the power board: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, J4 NTC 103AT on the cells, U2 BQ25798RQMR

Commit message: Combined power + charger project, charger schematic wired, 30 mm charger board
- hardware/power_charger_board: a copy of the power board with the charger
  added, for laying both out as one board. One schematic sheet (charger as
  section 4), charger parts on their own 22 x 30 mm outline beside the
  power board, the XT30s that linked the boards (J10, J11, J21, J22)
  removed, 4 copper layers, a Charger net class (3 mm) on PMID, SYS, SW1
  and SW2.
- Charger schematic (standalone and combined) redrawn with the parts wired
  to the BQ25798's pins; short two-pin nets now use KiCad's automatic
  names, renamed to match in the boards.
- Standalone charger board: 54 x 30 mm outline for the narrow enclosure,
  inductor pulled in, NTC connector moved; KXUSBC2 noted as a layout
  reference.
- Generator: can build one board; refuses the hand-edited power and
  charger boards unless forced; pre-defined track and via sizes.

Co-Authored-By: Claude Opus 5.5 <noreply@anthropic.com>
Claude-Session: https://claude.ai/code/session_01UUhpevE9ZSCJvyu3edQmf9
Connections:
- net BATP: no longer names the net of R11.1, U2.18 (BATP)
- net BTST1: no longer names the net of C26.1, U2.4 (BTST1)
- net BTST2: no longer names the net of C27.1, U2.19 (BTST2)
- net CHG_CE: no longer names the net of R14.1, U2.13 (CE_N)
- net CHG_ILIM: no longer names the net of R37.2, R38.1, U2.17 (ILIM_HIZ)
- net CHG_PROG: no longer names the net of R10.1, U2.20 (PROG)
- net CHG_STAT: no longer names the net of LED1.1 (C), U2.1 (STAT)
- net CHG_TS: no longer names the net of J4.1, R12.2, R13.1, U2.16 (TS)
- net SDRV: no longer names the net of C28.1, U2.24 (SDRV)
- net STAT_LED: no longer names the net of LED1.2 (A), R15.2
Other:
- moved on the sheet: C10, C11, C12, C13, C14, C15, C16, C17, C18, C19, C20, C21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
