File: hardware/power_charger_board/kicad/nibbles_power_charger.kicad_sch (KiCad schematic)
At the start: 95 parts, among them J12 JST-GH 6 (charger port: I2C), J2 XT30PW-M (dock power, from th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, J23 JST-GH 6 (to the power board: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, J3 XT30 (pack, from 4S BMS), J4 NTC 103AT on the cells, J5 XT30 (to the 5 V lighting con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, J6 To the base board (JST-GH 8), J7 S3B-PH-K-S (dock data, from t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, J8 S2B-PH-K-S (dock LED, panel), J9 JST-GH 6 (keypad port: I2C), Q5 30V N-FET >= 15 A, Q6 30V N-FET >= 15 A, Q7 2N7002, Q8 2N7002, Q9 30V N-FET >= 15 A, U2 BQ25798RQMR, U3 LM74700-Q1 (dock), U4 LM74700-Q1 (pack), U5 TPS259827ONRGET, U6 INA226AIDGSR, U7 TPS62933DRLR, U8 TCA9534PWR, U9 LM74700-Q1 (LEMO)

Commit message: Power + charger board: KXUSBC2 charger layout, test points, J6 fix, layout routed
- Charger section copied from KXUSBC2's BQ25792 layout (placement, tracks,
  vias, zones), KX-only parts dropped; R10-R13/C28 to 0402; dock input
  snubber R39/C49/C50; minimums relaxed to JLCPCB/KX values
- J6 footprint corrected (board top faces the 3.49's battery side, screen
  up), its holes on User.Drawings, 3D model 11 mm up; D5 to A11 and
  DOCK_DET to A6, R3 to B6
- Connectors all vertical JST-GH; J12/J23 removed; J10 (GH8 cable to the
  3.49) and J11 (second I2C port) added; H1-H3 M2.5 holes; connector
  labels and board name
- Test points TP3-TP24 on the bottom; CHG_ILIM and EFUSE_IMON named
- Schematic: DOCK_DATA_RAW/DOCK_DET_RAW short removed, C30 pins matched
- Routing by hand in KiCad (in progress; review findings still open)

Co-Authored-By: Claude Opus 5.5 <noreply@anthropic.com>
Claude-Session: https://claude.ai/code/session_01UUhpevE9ZSCJvyu3edQmf9
Parts:
- removed J12: JST-GH 6 (charger port: I2C), Connector_JST:JST_GH_SM06B-GHS-TB_1x06-1MP_P1.25mm_Horizontal, symbol nibbles:CONN6
- removed J23: JST-GH 6 (to the power board: I2C), Connector_JST:JST_GH_SM06B-GHS-TB_1x06-1MP_P1.25mm_Horizontal, symbol nibbles:CONN6
- added C49, C50: 1uF 50V, Capacitor_SMD:C_0603_1608Metric, symbol nibbles:C
- added D5: SS34, Diode_SMD:D_SMA, symbol nibbles:D
- added J10: JST-GH 8 vertical (cable to the 3.49, instead of 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, Connector_JST:JST_GH_BM08B-GHS-TBT_1x08-1MP_P1.25mm_Vertical, symbol nibbles:CONN8
- added J11: JST-GH 6 vertical (I2C port 2: pole segment), Connector_JST:JST_GH_BM06B-GHS-TBT_1x06-1MP_P1.25mm_Vertical, symbol nibbles:CONN6
- added R39: 2 (input snubber), Resistor_SMD:R_0603_1608Metric, symbol nibbles:R
- added TP1: GND, TestPoint:TestPoint_Pad_2.5x2.5mm, symbol Connector:TestPoint
- added TP10: +5V, TestPoint:TestPoint_Pad_D1.5mm, symbol Connector:TestPoint
- added TP11: +3V3, TestPoint:TestPoint_Pad_D1.5mm, symbol Connector:TestPoint
- added TP12: SYS, TestPoint:TestPoint_Pad_D1.5mm, symbol Connector:TestPoint
- added TP13: PMID, TestPoint:TestPoint_Pad_D1.5mm, symbol Connector:TestPoint
- added TP14: REGN, TestPoint:TestPoint_Pad_D1.5mm, symbol Connector:TestPoint
- added TP15: EFUSE_IMON, TestPoint:TestPoint_Pad_D1.5mm, symbol Connector:TestPoint
- added TP16: CHG_ILIM, TestPoint:TestPoint_Pad_D1.5mm, symbol Connector:TestPoint
- added TP17: EFUSE_PG, TestPoint:TestPoint_Pad_D1.5mm, symbol Connector:TestPoint
- added TP18: EFUSE_EN, TestPoint:TestPoint_Pad_D1.5mm, symbol Connector:TestPoint
- added TP19: GATE_DOCK, TestPoint:TestPoint_Pad_D1.5mm, symbol Connector:TestPoint
- added TP2: TS, TestPoint:TestPoint_Pad_2.5x2.5mm, symbol Connector:TestPoint
- added TP20: GATE_PACK, TestPoint:TestPoint_Pad_D1.5mm, symbol Connector:TestPoint
- added TP21: GATE_LEMO, TestPoint:TestPoint_Pad_D1.5mm, symbol Connector:TestPoint
- added TP22: CHG_QON, TestPoint:TestPoint_Pad_D1.5mm, symbol Connector:TestPoint
- added TP23: DOCK_DET, TestPoint:TestPoint_Pad_D1.5mm, symbol Connector:TestPoint
- added TP24: DOCK_UART, TestPoint:TestPoint_Pad_D1.5mm, symbol Connector:TestPoint
- added TP3, TP4: GND, TestPoint:TestPoint_Pad_D1.5mm, symbol Connector:TestPoint
- added TP5: DOCK_RAW, TestPoint:TestPoint_Pad_D1.5mm, symbol Connector:TestPoint
- added TP6: DOCK_VIN, TestPoint:TestPoint_Pad_D1.5mm, symbol Connector:TestPoint
- added TP7: PACK_F, TestPoint:TestPoint_Pad_D1.5mm, symbol Connector:TestPoint
- added TP8: LIGHT_BUS, TestPoint:TestPoint_Pad_D1.5mm, symbol Connector:TestPoint
- added TP9: LIGHT_OUT, TestPoint:TestPoint_Pad_D1.5mm, symbol Connector:TestPoint
- C28: footprint Capacitor_SMD:C_0603_1608Metric -> Capacitor_SMD:C_0402_1005Metric
- J4: value NTC 103AT on the cells -> NTC 103AT on the cells (JST-GH 2, vertical); footprint Connector_JST:JST_PH_S2B-PH-K_1x02_P2.00mm_Horizontal -> Connector_JST:JST_GH_BM02B-GHS-TBT_1x02-1MP_P1.25mm_Vertical; LCSC C173752 -> (none); MPN S2B-PH-K-S -> BM02B-GHS-TBT
- J6: value To the base board (JST-GH 8) -> To the 3.49 (stacked headers); footprint Connector_JST:JST_GH_SM08B-GHS-TB_1x08-1MP_P1.25mm_Horizontal -> nibbles:Waveshare_ESP32-S3-Touch-LCD-3.49_Headers; symbol nibbles:CONN8 -> nibbles:WS_ESP32S3_LCD349_HDR; LCSC C265111 -> (none); MPN SM08B-GHS-TB -> 2x 1x11 female header, 2.54 mm
- J7: value S3B-PH-K-S (dock data, from the LEMO) -> BM02B-GHS-TBT (dock data + detect, from the LEMO); footprint Connector_JST:JST_PH_S3B-PH-K_1x03_P2.00mm_Horizontal -> Connector_JST:JST_GH_BM02B-GHS-TBT_1x02-1MP_P1.25mm_Vertical; symbol nibbles:CONN3 -> nibbles:CONN2_PH2; LCSC C157929 -> (none); MPN S3B-PH-K-S -> BM02B-GHS-TBT
- J8: value S2B-PH-K-S (dock LED, panel) -> BM02B-GHS-TBT (dock LED, panel); footprint Connector_JST:JST_PH_S2B-PH-K_1x02_P2.00mm_Horizontal -> Connector_JST:JST_GH_BM02B-GHS-TBT_1x02-1MP_P1.25mm_Vertical; LCSC C173752 -> (none); MPN S2B-PH-K-S -> BM02B-GHS-TBT
- J9: value JST-GH 6 (keypad port: I2C) -> JST-GH 6 vertical (keypad port: I2C); footprint Connector_JST:JST_GH_SM06B-GHS-TB_1x06-1MP_P1.25mm_Horizontal -> Connector_JST:JST_GH_BM06B-GHS-TBT_1x06-1MP_P1.25mm_Vertical; MPN SM06B-GHS-TB -> BM06B-GHS-TBT
- R10, R11, R12, R13: footprint Resistor_SMD:R_0603_1608Metric -> Resistor_SMD:R_0402_1005Metric
Connections:
- net +3V3: now also J6.A10 (3V3), J6.B10 (3V3), J10.3, J11.2, TP11.1; no longer J6.3
- net +5V: now also D5.2 (A), J11.6, TP10.1; no longer J6.1
- net CHG_QON: now also TP22.1
- net DOCK_DET: now also J6.A6 (IO5), J10.8, TP23.1; no longer J6.8
- net DOCK_RAW: now also R39.2, TP5.1
- net DOCK_UART: now also J6.B6 (IO44), J10.7, TP24.1; no longer J6.7
- net DOCK_VIN: now also TP6.1
- net EFUSE_EN: now also TP18.1
- net EFUSE_PG: now also TP17.1
- net GATE_DOCK: now also TP19.1
- net GATE_LEMO: now also TP21.1
- net GATE_PACK: now also TP20.1
- net GND: now also J6.A9 (GND), J6.B9 (GND), C49.1, C50.1, J10.2, J11.1, TP1.1, TP3.1, TP4.1; no longer J6.2, J7.3
- net LIGHT_BUS: now also TP8.1
- net LIGHT_OUT: now also TP9.1
- net PACK_F: now also TP7.1
- net PMID: now also TP13.1
- net PWR_INT: now also J6.A4 (IO3), J10.6, J11.5; no longer J6.6
- net PWR_SCL: now also J6.A3 (IO2), J10.5, J11.4; no longer J6.5
- net PWR_SDA: now also J6.A2 (IO1), J10.4, J11.3; no longer J6.4
- net REGN: now also TP14.1
- net SYS: now also TP12.1
- net CHG_ILIM: now reaches R37.2, R38.1, U2.17 (ILIM_HIZ)
- net CHG_ILIM: now also TP16.1
- net CHG_TS: now reaches J4.1, R12.2, R13.1, U2.16 (TS)
- net CHG_TS: now also TP2.1
- net EFUSE_IMON: now reaches R27.1, U5.9 (IMON)
- net EFUSE_IMON: now also TP15.1
- new net: C49.2, C50.2, R39.1
- new net +5V_349: D5.1 (C), J10.1, J6.A11 (5V)
- no-connect marks 9 -> 21
Other:
- note added: "Test points: bottom side, bare 1.5 mm pads (TP1 GND and TP2 TS are the 2.5 mm ones by the charger)"
- note added: "pins (LEMO 1-3 +, 4-6 ground), J7 (JST-GH 2) its data (LEMO 7, UART to the base) and dock detect (8)."
- note removed: "pins (LEMO 1-3 +, 4-6 ground), J7 (JST-PH 3) its data (LEMO 7, UART to the base), dock detect (8) and a ground."
- moved on the sheet: C30, C48, D2, D3, D4, J2, Q9, R3, R35, R5, U9

Commit message: Power + charger board: JLCPCB fab files, LCSC and DigiKey orders
- fab/export.sh: gerbers, drills, JLCPCB BOM/CPL after ERC, DRC and parity
  checks, plus LCSC and DigiKey order lists (DigiKey parts from
  digikey_map.csv; what DigiKey can't supply goes to an LCSC gaps list)
- LCSC fields on every part, picked to be in stock at LCSC for a hand build
- eFuse timing caps set: C35 ITIMER 22n, C36 RETRY_DLY 22n, C37 dVdt 47n;
  R27 IMON 1k

Co-Authored-By: Claude Opus 5.5 <noreply@anthropic.com>
Claude-Session: https://claude.ai/code/session_01UUhpevE9ZSCJvyu3edQmf9
Parts:
- C12, C16, C22: LCSC (none) -> C131394
- C25: LCSC (none) -> C19666
- C26, C27: LCSC (none) -> C1622
- C28: LCSC (none) -> C106205
- C30, C31, C38, C42, C43, C47, C48: LCSC (none) -> C14663
- C35: value 10nF (TBD) -> 22nF; LCSC (none) -> C21122
- C36: value 100nF (TBD) -> 22nF; LCSC (none) -> C21122
- C37: value 22nF (TBD) -> 47nF; LCSC (none) -> C1622
- C40, C41: LCSC (none) -> C89632
- C44, C45: LCSC (none) -> C45783
- C46: LCSC (none) -> C1589
- C49, C50: LCSC (none) -> C15849
- J10: LCSC (none) -> C133062
- J11, J9: LCSC (none) -> C189892
- J4, J7, J8: LCSC (none) -> C161690
- J6: LCSC (none) -> C2932674
- L1: LCSC C408445 -> C285810
- L2: LCSC C408449 -> C285805
- R10: LCSC (none) -> C25771
- R11: LCSC (none) -> C25076
- R12: LCSC (none) -> C2933105
- R13: LCSC (none) -> C2998131
- R14, R16, R24, R28, R31, R37: LCSC (none) -> C98220
- R15: LCSC (none) -> C4190
- R20, R21, R35: LCSC (none) -> C22935
- R22, R25, R5: LCSC (none) -> C25803
- R23: LCSC (none) -> C23121
- R26: LCSC (none) -> C22796
- R27: value TBD (IMON) -> 1k; LCSC (none) -> C21190
- R3, R4: LCSC (none) -> C21190
- R30: LCSC (none) -> C2933235
- R32, R33: LCSC (none) -> C23162
- R36: LCSC (none) -> C23234
- R38: LCSC (none) -> C22857
- R39: LCSC (none) -> C22977
Other:
- note added: "dVdt 47n: 170 ms ramp, under 2.5 W start-up heating up to ~2 mF on EFUSE_OUT. ITIMER 22n: 10 ms overload blanking. RETRY_DLY 22n: retry after 1 s."
- note removed: "ITIMER, RETRY_DLY and dVdt values are starting points: check against the datasheet for the converter's input capacitance."
